File: cape_op-amp.kicad_pcb (KiCad board)
At the start: 2 copper layers, 123.6 x 99.6 mm, 12 parts, among them J1 Conn_01x01_Socket, J2 Conn_01x01_Socket, J3 Conn_01x01_Socket, J4 Conn_01x01_Socket, U1 LM741

Commit message: added github link to readme
Other:
- board text added: "CAPE Physics Unit 2 Workshop Operational Amplifiers UWI Mona https://github.com/irpl/cape_op-amp"
- board text removed: "CAPE Physics Unit 2 Workshop Operational Amplifiers UWI Mona"
Changed lines of the file:
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@@
 		)
 	)
-	(gr_text "CAPE Physics\nUnit 2 Workshop\nOperational Amplifiers\nUWI Mona"
+	(gr_text "CAPE Physics\nUnit 2 Workshop\nOperational Amplifiers\nUWI Mona\nhttps://github.com/irpl/cape_op-amp"
 		(at 85 117.5 0)
 		(layer "F.SilkS")
